File: hardware/mpu6050_board/mpu6050_board.kicad_sch (KiCad schematic)
At the start: 0 parts

Commit message: Update schematic (ERC clean), remove KiCad temp files
Parts:
- added A1: Arduino_Nano_v3.x, Module:Arduino_Nano, symbol MCU_Module:Arduino_Nano_v3.x
- added J1: GY-521 (MPU6050), symbol Connector_Generic:Conn_01x08
Connections:
- new net +5V: A1.27 (+5V), J1.VCC (Pin_1)
- new net GND: A1.29 (GND), A1.4 (GND), J1.AD0 (Pin_7), J1.GND (Pin_2)
- new net SCL: A1.24 (A5), J1.SCL (Pin_3)
- new net SDA: A1.23 (A4), J1.SDA (Pin_4)
- no-connect marks 0 -> 6
Other:
- title: (none) -> MPU6050 + Arduino Nano Sensor Board
